File: hardware/kicad-project/fixedwing-fcu.kicad_sch (KiCad schematic)
At the start: 0 parts

Commit message: added mounting hole and tentative MCU
Parts:
- added H1: MountingHole_M3_3.2mm_Pad, PCM_SL_Mechanical:MountingHole_3.2mm_Pad, symbol PCM_SL_Mechanical:MountingHole_M3_3.2mm_Pad
- added U1: STM32F401CCUx, Package_DFN_QFN:QFN-48-1EP_7x7mm_P0.5mm_EP5.6x5.6mm, symbol MCU_ST_STM32F4:STM32F401CCUx
Connections:
- new net: U1.23 (VSS), U1.35 (VSS), U1.47 (VSS), U1.49 (VSS)
Changed lines of the file:
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@@
 	(generator_version "9.0")
 	(paper "A4")
+	(symbol
+		(lib_id "MCU_ST_STM32F4:STM32F401CCUx")
+		(at 186.69 85.09 0)
+		(unit 1)
+		(exclude_from_sim no)
+		(in_bom yes)
+		(on_board yes)
+		(dnp no)
+		(fields_autoplaced yes)
+		(property "Reference" "U1"
+			(at 191.3733 128.27 0)
+			(effects
+				(font
+					(size 1.27 1.27)
+				)
+				(justify left)
+			)
+		)
+		(property "Value" "STM32F401CCUx"
+			(at 191.3733 130.81 0)
+			(effects
+				(font
+					(size 1.27 1.27)
+				)
+				(justify left)
+			)
+		)
+		(property "Footprint" "Package_DFN_QFN:QFN-48-1EP_7x7mm_P0.5mm_EP5.6x5.6mm"
+			(at 173.99 125.73 0)
+			(effects
+				(font
+					(size 1.27 1.27)
+				)
+				(justify right)
+				(hide yes)
+			)
+		)
+		(property "Datasheet" "https://www.st.com/resource/en/datasheet/stm32f401cc.pdf"
+			(at 186.69 85.09 0)
+			(effects
+				(font
+					(size 1.27 1.27)
+				)
+				(hide yes)
+			)
+		)
+		(property "Description" "STMicroelectronics Arm Cortex-M4 MCU, 256KB flash, 64KB RAM, 84 MHz, 1.7-3.6V, 36 GPIO, UFQFPN48"
+			(at 186.69 85.09 0)
+			(effects
+				(font
+					(size 1.27 1.27)
+				)
+				(hide yes)
+			)
+		)
+		(pin "39"
+		)
+		(pin "36"
+		)
+		(pin "20"
+		)
+		(pin "11"
+		)
+		(pin "6"
+		)
+		(pin "12"
+		)
+		(pin "34"
+		)
+		(pin "13"
+		)
+		(pin "28"
+		)
+		(pin "37"
+		)
+		(pin "24"
+		)
+		(pin "8"
+		)
+		(pin "44"
+		)
+		(pin "15"
+		)
+		(pin "4"
+		)
+		(pin "38"
+		)
+		(pin "31"
+		)
+		(pin "18"
+		)
+		(pin "5"
+		)
+		(pin "19"
+		)
+		(pin "2"
+		)
+		(pin "3"
+		)
+		(pin "21"
+		)
+		(pin "16"
+		)
+		(pin "9"
+		)
+		(pin "46"
+		)
+		(pin "45"
+		)
+		(pin "7"
+		)
+		(pin "29"
+		)
+		(pin "23"
+		)
+		(pin "42"
+		)
+		(pin "43"
+		)
+		(pin "32"
+		)
+		(pin "14"
+		)
+		(pin "47"
+		)
+		(pin "49"
+		)
+		(pin "10"
+		)
+		(pin "40"
+		)
+		(pin "27"
+		)
+		(pin "1"
+		)
+		(pin "35"
+		)
+		(pin "30"
+		)
+		(pin "22"
+		)
+		(pin "41"
+		)
+		(pin "33"
+		)
+		(pin "48"
+		)
+		(pin "25"
+		)
+		(pin "17"
+		)
+		(pin "26"
+		)
+		(instances
+			(project ""
+				(path "/ac0c94ab-76b3-44d5-8ba2-dc5bdbe4c28a"
+					(reference "U1")
+					(unit 1)
+				)
+			)
+		)
+	)
+	(symbol
+		(lib_id "PCM_SL_Mechanical:MountingHole_M3_3.2mm_Pad")
+		(at 111.76 82.55 0)
+		(unit 1)
+		(exclude_from_sim no)
+		(in_bom yes)
+		(on_board yes)
+		(dnp no)
+		(fields_autoplaced yes)
+		(property "Reference" "H1"
+			(at 115.57 81.2799 0)
+			(effects
+				(font
+					(size 1.27 1.27)
+				)
+				(justify left)
+			)
+		)
+		(property "Value" "MountingHole_M3_3.2mm_Pad"
+			(at 115.57 83.8199 0)
+			(effects
+				(font
+					(size 1.27 1.27)
+				)
+				(justify left)
+			)
+		)
+		(property "Footprint" "PCM_SL_Mechanical:MountingHole_3.2mm_Pad"
+			(at 111.76 86.36 0)
+			(effects
+				(font
+					(size 1.27 1.27)
+				)
+				(hide yes)
+			)
+		)
+		(property "Datasheet" ""
+			(at 111.76 82.55 0)
+			(effects
+				(font
+					(size 1.27 1.27)
+				)
+				(hide yes)
+			)
+		)
+		(property "Description" "3.2mm Diameter Mounting Hole Pad (M3)"
+			(at 111.76 82.55 0)
+			(effects
+				(font
+					(size 1.27 1.27)
+				)
+				(hide yes)
+			)
+		)
+		(pin "1"
+		)
+		(instances
+			(project ""
+				(path "/ac0c94ab-76b3-44d5-8ba2-dc5bdbe4c28a"
+					(reference "H1")
+					(unit 1)
+				)
+			)
+		)
+	)
 	(sheet_instances
 		(path "/"
